Commit message: Собрал контейнеры (есть проблемы)

File: urdf/common_macro.xacro (robot description, xacro)
@@ -1,14 +1,4 @@
 <?xml version="1.0"?>
 <robot name="dron_macro" xmlns:xacro="http://www.ros.org/wiki/xacro">
-<!-- *********************************************************************** -->
-<!-- Macro for cylinder inertial model -->
-<xacro:macro name="cylinder_inertia" params ="m r h">
-  <inertial>
-   <mass value="${m}"/> <!-- Cylinder mass -->
-   <!-- Formulas to calculate inertia moments for cylinder -->
-   <inertia ixx="${m*(3*r*r+h*h)/12}"  ixy="0.0" ixz="0.0"
-            iyy="${m*(3*r*r+h*h)/12}"  iyz="0.0" izz="${m*r*r/2}"/>
-   </inertial>
-</xacro:macro>
 <!-- *********************************************************************** -->
 <!-- Macro for base inertial model -->
@@ -33,4 +23,5 @@
     </inertial>
 </xacro:macro>
+<!-- Macro for box inertial model -->
 <xacro:macro name="inertial_box" params="mass x y z">
     <inertial>
@@ -41,4 +32,5 @@
     </inertial>
 </xacro:macro>
+<!-- Macro for cylinder inertial model -->
 <xacro:macro name="inertial_cylinder" params="mass length radius">
     <inertial>

File: urdf/dron_base.xacro (robot description, xacro)
@@ -78,5 +78,5 @@
   <xacro:motor name="rear_right_motor" mass="${motor_mass}" length="${motor_length}" radius="${motor_radius}" color="${motor_color}" origin="${motor_offset_x} -${motor_offset_y} 0"/>
   <gazebo>
-    <plugin name="gazebo_ros_control" filename="libgazebo_ros_control.so">
+    <plugin name="ros_gz_control" filename="libros_gz_control.so">
         <robotNamespace>/</robotNamespace>
     </plugin>
